Commit message: Sync M2/M3 work: real-map SLAM pipeline on Modal, ICP loop closure fix, canonical interface contracts, src/ reorg

File: src/simulation/rambla_description/urdf/params.xacro (robot description, xacro)
@@ -15,14 +15,32 @@
   <xacro:property name="base_diameter" value="0.349"/>
   <xacro:property name="wheel_base" value="0.235"/>
-  <!-- Body cylinder: top is 79mm above the floor, minus 12.5mm floor gap = 66.5mm tall.
-       LiDAR housing sits on top (body top 79mm + 18mm housing = ~97mm total height). -->
+  <!-- Body cylinder: top is 79mm above the floor, minus 12.5mm floor gap = 66.5mm tall. -->
   <xacro:property name="lower_cylinder_height" value="0.0665"/>
-  <!-- LiDAR housing, 18mm, seated flush on the body top -->
+  <!-- LiDAR housing, 18mm tall. -->
   <xacro:property name="laser_puck_height" value="0.018"/>
   <xacro:property name="laser_puck_diameter" value="0.083"/>
-  <!-- offset = laser_puck_height/2 so the housing bottom sits at the body top -->
-  <xacro:property name="laser_puck_offset" value="0.009"/>
+  <!-- Scan-plane height above the body top (M1, PHY-004 sensor-placement
+       revisit): the scan plane sits at lower_cylinder_height + this offset
+       in base_link frame. Previously 0.009 (= laser_puck_height/2, housing
+       flush on the body top) put the plane at z=0.0755, which cuts directly
+       through the forward camera box (camera_z +/- camera_height/2 =
+       [0.065, 0.085] - see camera_z comment below) at x=0.1545..0.1745,
+       ~0.251-0.271m from the rear-offset LiDAR - this is the forward
+       self-return documented in rambla_safety's min_valid_range_m (that
+       doc's "sees its own front bumper" wording is inaccurate: the bumper's
+       z-band [0.008, 0.058] never reaches the scan plane at all; verified by
+       direct calculation, the camera is the actual obstruction). Raised to
+       0.0335 so the scan plane (z=0.10) clears the camera top (0.085) by
+       15mm - eliminates the forward self-return rather than just filtering
+       it. Placeholder cosmetic note: this puts the housing ~24.5mm above the
+       body top with no mast geometry filling the gap (a small floating-turret
+       look) - acceptable for this placeholder-grade body (PHY-004); revisit
+       with a real mount at M10/M11. -->
+  <xacro:property name="laser_puck_offset" value="0.0335"/>
   <!-- LiDAR turret sits toward the REAR of the body, not centered. +X is forward,
-       so negative shifts it back. -->
+       so negative shifts it back. Left as-is by the M1 sensor-placement revisit -
+       the vertical raise above fully resolves the forward self-detection
+       regardless of this offset, and rambla_safety's front-arc check only looks
+       forward, so the rear placement doesn't affect stop-distance behavior. -->
   <xacro:property name="lidar_center_offset" value="-0.0965"/>
   <!-- N*m -->
@@ -37,10 +55,18 @@
        spans 0..+90 deg, right half -90..0 deg (they meet at the front, 0 deg, so
        there is no dead-center gap). Each half is its own dedicated link (bumper_left,
-       bumper_right) with exactly one unnamed collision spanning its 90 deg arc as a
-       single box - one sensor watching one collision per link, matching the proven
-       working pattern in iRobotEducation/create3_sim rather than the many
-       named-facet-collisions-per-sensor layout this replaced (see
-       bugs/bumper-contact-sensor-silent.md). Bumper sits at the body radius and
-       protrudes a few mm so it's the surface that touches obstacles. -->
+       bumper_right) with exactly one unnamed collision - one sensor watching one
+       collision per link, matching the proven working pattern in
+       iRobotEducation/create3_sim rather than the many named-facet-collisions-
+       per-sensor layout this replaced (see bugs/bumper-contact-sensor-silent.md).
+       As of M1 (SIM-003/PHY-004), each half's collision+visual is a solid
+       circular-segment MESH (see meshes/generate_bumper_mesh.py and the
+       bumper_half macro in rambla.urdf.xacro) whose outer face follows the true
+       body radius all the way around its 90 deg arc, rather than the old
+       single flat box per half that protruded ~5cm past the body at the front
+       centerline (audit 2026-07-08-accepted-stabilization-findings.md §3/P1-1).
+       bumper_thickness/bumper_height still set the mesh's radial thickness and
+       vertical band; bumper_z is still its mount height. Bumper sits at the
+       body radius and protrudes a few mm so it's the surface that touches
+       obstacles. -->
   <xacro:property name="bumper_thickness" value="0.010"/> <!-- radial; outer face ~5mm proud -->
   <xacro:property name="bumper_height" value="0.050"/>

File: src/simulation/rambla_description/urdf/rambla.urdf.xacro (robot description, xacro)
@@ -6,20 +6,27 @@
   <xacro:include filename="materials.xacro" />
   <!-- ****************** **************** ****************** -->
-  <!-- One bumper half: a single box spanning its 90-deg arc (midpoint angle
-       a0+45), tangent to the body at the body radius. Exactly one unnamed
-       collision per link (sdformat auto-names it "<link>_collision") so the
-       contact sensor watches one collision on its own dedicated link - the
-       pattern proven working in iRobotEducation/create3_sim, replacing the
-       many-named-facet-collisions-per-sensor layout this repo used to have. -->
-  <xacro:macro name="bumper_half" params="name parent a0">
-    <xacro:property name="ang" value="${a0 + 45}"/>
-    <!-- Chord of the full 90-deg arc, padded 15% so it comfortably covers the
-         arc's midpoint tangent without falling short at the edges. -->
-    <xacro:property name="width" value="${2 * (base_diameter/2) * sin(0.5 * 90.0 * DEG2RAD) * 1.15}"/>
+  <!-- One bumper half: a solid circular-segment mesh (outer arc at the body
+       radius + a single straight closing chord - convex by construction,
+       since a chord-closed arc under 180 deg is always convex regardless of
+       facet count) following the body's true circular shape, replacing the
+       old single-flat-box-per-half wedge that protruded ~5cm past the body
+       at the front centerline (see README.md M1 /
+       .claude/internal-docs/audits/2026-07-08-accepted-stabilization-findings.md
+       §3/P1-1). Convexity matters here specifically because it makes the
+       mesh immune to a physics engine silently substituting a convex hull
+       or convex decomposition for a non-static body's mesh collision - what
+       gets simulated is exactly what was authored either way. Meshes are
+       generated by meshes/generate_bumper_mesh.py directly in base_link-frame
+       absolute angles (bumper_left = 0..+90 deg, bumper_right = -90..0 deg),
+       so the joint origin below is a straight translation to the bumper
+       band height with no rotation. Exactly one unnamed collision per link
+       (sdformat auto-names it "<link>_collision") so the contact sensor
+       watches one collision on its own dedicated link - the pattern proven
+       working in iRobotEducation/create3_sim, unchanged by this mesh swap. -->
+  <xacro:macro name="bumper_half" params="name parent mesh">
     <joint name="${name}_joint" type="fixed">
       <parent link="${parent}"/>
       <child link="${name}"/>
-      <origin xyz="${(base_diameter/2)*cos(ang*DEG2RAD)} ${(base_diameter/2)*sin(ang*DEG2RAD)} ${bumper_z}"
-              rpy="0 0 ${(ang+90)*DEG2RAD}"/>
+      <origin xyz="0 0 ${bumper_z}" rpy="0 0 0"/>
     </joint>
     <gazebo reference="${name}_joint">
@@ -30,5 +37,5 @@
         <origin xyz="0 0 0" rpy="0 0 0"/>
         <geometry>
-          <box size="${width} ${bumper_thickness} ${bumper_height}"/>
+          <mesh filename="package://rambla_description/meshes/${mesh}"/>
         </geometry>
         <material name="dark"/>
@@ -37,8 +44,11 @@
         <origin xyz="0 0 0" rpy="0 0 0"/>
         <geometry>
-          <box size="${width} ${bumper_thickness} ${bumper_height}"/>
+          <mesh filename="package://rambla_description/meshes/${mesh}"/>
         </geometry>
       </collision>
-      <xacro:solid_box_inertia m="0.02" x="${width}" y="${bumper_thickness}" z="${bumper_height}"/>
+      <xacro:solid_box_inertia m="0.02"
+        x="${(base_diameter/2)+(bumper_thickness/2)}"
+        y="${(base_diameter/2)+(bumper_thickness/2)}"
+        z="${bumper_height}"/>
     </link>
   </xacro:macro>
@@ -85,7 +95,9 @@
   <!-- Front bumper = front 180 deg of the body, as two dedicated links (each
        with its own fixed joint + single collision). Left half 0..+90 deg,
-       right half -90..0 deg (meet at the front, 0 deg, no dead-center gap). -->
-  <xacro:bumper_half name="bumper_left" parent="base_link" a0="0"/>
-  <xacro:bumper_half name="bumper_right" parent="base_link" a0="-90"/>
+       right half -90..0 deg (meet at the front, 0 deg, no dead-center gap).
+       Each mesh already encodes its own absolute angular range - see the
+       bumper_half macro comment above. -->
+  <xacro:bumper_half name="bumper_left" parent="base_link" mesh="bumper_left.stl"/>
+  <xacro:bumper_half name="bumper_right" parent="base_link" mesh="bumper_right.stl"/>
   <joint name="caster_joint" type="fixed">
     <parent link="base_link"/>
